File: PCB/launchpad.kicad_pcb (KiCad board)
At the start: 2 copper layers, 100 x 100 mm, 39 parts, among them SW1 Kaihua PG1350, SW10 Kaihua PG1350, SW11 Kaihua PG1350, SW12 Kaihua PG1350, SW13 PEC11R-4220F-S0012, SW2 Kaihua PG1350, SW3 Kaihua PG1350, SW4 Kaihua PG1350, SW5 Kaihua PG1350, SW6 Kaihua PG1350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

Commit message: R1 sent to fab
Parts:
- LED1, LED10, LED11, LED12, LED13, LED2, LED3, LED4, LED9: value WS2812B-4020 -> XL-3528RGBW-WS2812B; footprint easyeda_kicad:LED-SMD_WS2812B-4020 -> 1_easyeda_kicad:LED-SMD_4P-L3.5-W2.8-BR-1
- LED5: renamed from LED8; value WS2812B-4020 -> XL-3528RGBW-WS2812B; footprint easyeda_kicad:LED-SMD_WS2812B-4020 -> 1_easyeda_kicad:LED-SMD_4P-L3.5-W2.8-BR-1
- LED6: renamed from LED7; value WS2812B-4020 -> XL-3528RGBW-WS2812B; footprint easyeda_kicad:LED-SMD_WS2812B-4020 -> 1_easyeda_kicad:LED-SMD_4P-L3.5-W2.8-BR-1
- LED7: renamed from LED6; value WS2812B-4020 -> XL-3528RGBW-WS2812B; footprint easyeda_kicad:LED-SMD_WS2812B-4020 -> 1_easyeda_kicad:LED-SMD_4P-L3.5-W2.8-BR-1
- LED8: renamed from LED5; value WS2812B-4020 -> XL-3528RGBW-WS2812B; footprint easyeda_kicad:LED-SMD_WS2812B-4020 -> 1_easyeda_kicad:LED-SMD_4P-L3.5-W2.8-BR-1
- moved LED5 63.0 mm to (128.0, 116.3)
- moved LED8 63.0 mm to (191.0, 116.3)
- moved LED6 21.0 mm to (149.0, 116.3)
- moved LED7 21.0 mm to (170.0, 116.3)
- moved LED13 0.92 mm to (140.2, 60.2)
- moved D1 0.89 mm to (145.7, 61.0)
- moved LED1 0.70 mm to (128.0, 91.3)
- moved LED2 0.70 mm to (149.0, 91.3)
- moved LED3 0.70 mm to (170.0, 91.3)
- moved LED4 0.70 mm to (191.0, 91.3)
- moved LED10 0.70 mm to (149.0, 141.3)
- moved LED11 0.70 mm to (170.0, 141.3)
- moved LED12 0.70 mm to (191.0, 141.3)
- moved LED9 0.70 mm to (128.0, 141.3)
- moved R3 0.26 mm to (126.5, 58.5)
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Connections:
- LED1 pad 1: /NEOP -> GND
- LED1 pad 2: +5V -> /NEOP
- LED1 pad 3: Net-(LED1-Pad3) -> +5V
- LED1 pad 4: GND -> Net-(LED1-Pad4)
- LED10 pad 1: Net-(LED10-Pad1) -> GND
- LED10 pad 2: +5V -> Net-(LED10-Pad2)
- LED10 pad 3: Net-(LED10-Pad3) -> +5V
- LED10 pad 4: GND -> Net-(LED10-Pad4)
- LED11 pad 1: Net-(LED10-Pad3) -> GND
- LED11 pad 2: +5V -> Net-(LED10-Pad4)
- LED11 pad 3: Net-(LED11-Pad3) -> +5V
- LED11 pad 4: GND -> Net-(LED11-Pad4)
- LED12 pad 1: Net-(LED11-Pad3) -> GND
- LED12 pad 2: +5V -> Net-(LED11-Pad4)
- LED12 pad 3: unconnected-(LED12-Pad3) -> +5V
- LED12 pad 4: GND -> unconnected-(LED12-Pad4)
- LED13 pad 1: /NEOP1 -> GND
- LED13 pad 2: Net-(D1-Pad1) -> /NEOP1
- LED13 pad 3: /NEOP -> Net-(D1-Pad1)
- LED13 pad 4: GND -> /NEOP
- LED2 pad 1: Net-(LED1-Pad3) -> GND
- LED2 pad 2: +5V -> Net-(LED1-Pad4)
- LED2 pad 3: Net-(LED2-Pad3) -> +5V
- LED2 pad 4: GND -> Net-(LED2-Pad4)
- LED3 pad 1: Net-(LED2-Pad3) -> GND
- LED3 pad 2: +5V -> Net-(LED2-Pad4)
- LED3 pad 3: Net-(LED3-Pad3) -> +5V
- LED3 pad 4: GND -> Net-(LED3-Pad4)
- LED4 pad 1: Net-(LED3-Pad3) -> GND
- LED4 pad 2: +5V -> Net-(LED3-Pad4)
- LED4 pad 3: Net-(LED4-Pad3) -> +5V
- LED4 pad 4: GND -> Net-(LED4-Pad4)
- LED5 pad 1: Net-(LED4-Pad3) -> GND
- LED5 pad 2: +5V -> Net-(LED5-Pad2)
- LED5 pad 3: Net-(LED7-Pad1) -> +5V
- LED5 pad 4: GND -> Net-(LED9-Pad2)
- LED6 pad 1: Net-(LED7-Pad1) -> GND
- LED6 pad 2: +5V -> Net-(LED7-Pad4)
- LED6 pad 3: Net-(LED6-Pad1) -> +5V
- LED6 pad 4: GND -> Net-(LED5-Pad2)
- LED7 pad 1: Net-(LED6-Pad1) -> GND
- LED7 pad 2: +5V -> Net-(LED8-Pad4)
- LED7 pad 3: Net-(LED5-Pad1) -> +5V
- LED7 pad 4: GND -> Net-(LED7-Pad4)
- LED8 pad 1: Net-(LED5-Pad1) -> GND
- LED8 pad 2: +5V -> Net-(LED4-Pad4)
- LED8 pad 3: Net-(LED5-Pad3) -> +5V
- LED8 pad 4: GND -> Net-(LED8-Pad4)
- LED9 pad 1: Net-(LED5-Pad3) -> GND
- LED9 pad 2: +5V -> Net-(LED9-Pad2)
- LED9 pad 3: Net-(LED10-Pad1) -> +5V
- LED9 pad 4: GND -> Net-(LED10-Pad2)
Routing:
- net Net-(LED2-Pad4): track 0.00 -> 33.2 mm, vias 0 -> 2
- net Net-(LED2-Pad3): track 30.5 -> 0.00 mm, vias 2 -> 0
- net Net-(LED4-Pad3): track 28.1 -> 0.00 mm
- net Net-(LED10-Pad4): track 0.00 -> 27.8 mm, vias 0 -> 2
- net Net-(LED5-Pad3): track 27.6 -> 0.00 mm
- net Net-(LED3-Pad4): track 0.00 -> 27.4 mm, vias 0 -> 2
- net Net-(LED1-Pad4): track 0.00 -> 26.7 mm, vias 0 -> 2
- net Net-(LED10-Pad3): track 26.7 -> 0.00 mm, vias 2 -> 0
- net Net-(LED10-Pad2): track 0.00 -> 26.4 mm, vias 0 -> 2
- net Net-(LED9-Pad2): track 0.00 -> 26.0 mm
- net Net-(LED4-Pad4): track 0.00 -> 26.0 mm
- net Net-(LED11-Pad3): track 25.5 -> 0.00 mm, vias 2 -> 0
- net Net-(LED3-Pad3): track 25.4 -> 0.00 mm, vias 2 -> 0
- net Net-(LED10-Pad1): track 25.2 -> 0.00 mm, vias 2 -> 0
- net Net-(LED1-Pad3): track 25.0 -> 0.00 mm, vias 2 -> 0
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
Commit message: rename library
Parts:
- R1, R3: footprint easyeda_kicad:RES-ADJ-TH_RDC1022A05 -> 1_easyeda_kicad:RES-ADJ-TH_RDC1022A05
- R2: footprint easyeda_kicad:RES-TH_RK09K1130A6S -> 1_easyeda_kicad:RES-TH_RK09K1130A6S
- SW13: footprint easyeda_kicad:SW-TH_PEC11R-4220F-S0012 -> 1_easyeda_kicad:SW-TH_PEC11R-4220F-S0012
