File: PCB/launchpad.kicad_sch (KiCad schematic)
At the start: 39 parts, among them SW1 Kaihua PG1350, SW10 Kaihua PG1350, SW11 Kaihua PG1350, SW12 Kaihua PG1350, SW13 PEC11R-4220F-S0012, SW2 Kaihua PG1350, SW3 Kaihua PG1350, SW4 Kaihua PG1350, SW5 Kaihua PG1350, SW6 Kaihua PG1350, SW7 Kaihua PG1350, SW8 Kaihua PG1350, SW9 Kaihua PG1350, U1 RaspberryPi_Pico, U2 SSD1306

Commit message: R1 sent to fab
Parts:
- LED1, LED10, LED11, LED12, LED13, LED2, LED3, LED4, LED9: value WS2812B-4020 -> XL-3528RGBW-WS2812B; footprint easyeda_kicad:LED-SMD_WS2812B-4020 -> 1_easyeda_kicad:LED-SMD_4P-L3.5-W2.8-BR-1; symbol easyeda_kicad:WS2812B-4020 -> 1_easyeda_kicad:XL-3528RGBW-WS2812B; LCSC Part C965557 -> C2890364; Manufacturer Worldsemi -> XINGLIGHT(成兴光)
- LED5: renamed from LED8; value WS2812B-4020 -> XL-3528RGBW-WS2812B; footprint easyeda_kicad:LED-SMD_WS2812B-4020 -> 1_easyeda_kicad:LED-SMD_4P-L3.5-W2.8-BR-1; symbol easyeda_kicad:WS2812B-4020 -> 1_easyeda_kicad:XL-3528RGBW-WS2812B; LCSC Part C965557 -> C2890364; Manufacturer Worldsemi -> XINGLIGHT(成兴光)
- LED6: renamed from LED7; value WS2812B-4020 -> XL-3528RGBW-WS2812B; footprint easyeda_kicad:LED-SMD_WS2812B-4020 -> 1_easyeda_kicad:LED-SMD_4P-L3.5-W2.8-BR-1; symbol easyeda_kicad:WS2812B-4020 -> 1_easyeda_kicad:XL-3528RGBW-WS2812B; LCSC Part C965557 -> C2890364; Manufacturer Worldsemi -> XINGLIGHT(成兴光)
- LED7: renamed from LED6; value WS2812B-4020 -> XL-3528RGBW-WS2812B; footprint easyeda_kicad:LED-SMD_WS2812B-4020 -> 1_easyeda_kicad:LED-SMD_4P-L3.5-W2.8-BR-1; symbol easyeda_kicad:WS2812B-4020 -> 1_easyeda_kicad:XL-3528RGBW-WS2812B; LCSC Part C965557 -> C2890364; Manufacturer Worldsemi -> XINGLIGHT(成兴光)
- LED8: renamed from LED5; value WS2812B-4020 -> XL-3528RGBW-WS2812B; footprint easyeda_kicad:LED-SMD_WS2812B-4020 -> 1_easyeda_kicad:LED-SMD_4P-L3.5-W2.8-BR-1; symbol easyeda_kicad:WS2812B-4020 -> 1_easyeda_kicad:XL-3528RGBW-WS2812B; LCSC Part C965557 -> C2890364; Manufacturer Worldsemi -> XINGLIGHT(成兴光)
Connections:
- net +5V: now also LED1.3 (VDD), LED10.3 (VDD), LED11.3 (VDD), LED12.3 (VDD), LED2.3 (VDD), LED3.3 (VDD), LED4.3 (VDD), LED5.3 (VDD), LED6.3 (VDD), LED7.3 (VDD), LED8.3 (VDD), LED9.3 (VDD); no longer LED1.2 (VDD), LED10.2 (VDD), LED11.2 (VDD), LED12.2 (VDD), LED2.2 (VDD), LED3.2 (VDD), LED4.2 (VDD), LED5.2 (VDD), LED6.2 (VDD), LED7.2 (VDD), LED8.2 (VDD), LED9.2 (VDD)
- net GND: now also LED1.1 (VSS), LED10.1 (VSS), LED11.1 (VSS), LED12.1 (VSS), LED13.1 (VSS), LED2.1 (VSS), LED3.1 (VSS), LED4.1 (VSS), LED5.1 (VSS), LED6.1 (VSS), LED7.1 (VSS), LED8.1 (VSS), LED9.1 (VSS); no longer LED1.4 (VSS), LED10.4 (VSS), LED11.4 (VSS), LED12.4 (VSS), LED13.4 (VSS), LED2.4 (VSS), LED3.4 (VSS), LED4.4 (VSS), LED5.4 (VSS), LED6.4 (VSS), LED7.4 (VSS), LED8.4 (VSS), LED9.4 (VSS)
- net NEOP: now also LED1.2 (DIN), LED13.4 (DOUT); no longer LED1.1 (DIN), LED13.3 (DOUT)
- net NEOP1: now also LED13.2 (DIN); no longer LED13.1 (DIN)
- net at D1.1 (K): now also LED13.3 (VDD); no longer LED13.2 (VDD)
- new net: LED5.2 (DIN), LED6.4 (DOUT)
- new net: LED5.4 (DOUT), LED9.2 (DIN)
- new net: LED3.4 (DOUT), LED4.2 (DIN)
- new net: LED4.4 (DOUT), LED8.2 (DIN)
- new net: LED10.4 (DOUT), LED11.2 (DIN)
- new net: LED11.4 (DOUT), LED12.2 (DIN)
- new net: LED10.2 (DIN), LED9.4 (DOUT)
- new net: LED2.4 (DOUT), LED3.2 (DIN)
- new net: LED7.2 (DIN), LED8.4 (DOUT)
- new net: LED6.2 (DIN), LED7.4 (DOUT)
- new net: LED1.4 (DOUT), LED2.2 (DIN)

Commit message: rename library
Parts:
- R1, R3: footprint easyeda_kicad:RES-ADJ-TH_RDC1022A05 -> 1_easyeda_kicad:RES-ADJ-TH_RDC1022A05; symbol easyeda_kicad:RDC1022A05 -> 1_easyeda_kicad:RDC1022A05
- R2: footprint easyeda_kicad:RES-TH_RK09K1130A6S -> 1_easyeda_kicad:RES-TH_RK09K1130A6S; symbol easyeda_kicad:RK09K1130A6S -> 1_easyeda_kicad:RK09K1130A6S
- SW13: footprint easyeda_kicad:SW-TH_PEC11R-4220F-S0012 -> 1_easyeda_kicad:SW-TH_PEC11R-4220F-S0012; symbol easyeda_kicad:PEC11R-4220F-S0012 -> 1_easyeda_kicad:PEC11R-4220F-S0012
Changed lines of the file:
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@@
     (pin "2")
   )
-  (symbol (lib_id "easyeda_kicad:RK09K1130A6S") (at 66.04 184.15 90) (unit 1)
+  (symbol (lib_id "1_easyeda_kicad:RK09K1130A6S") (at 66.04 184.15 90) (unit 1)
     (in_bom yes) (on_board yes)
     (property "Reference" "R2" (id 0) (at 69.85 181.61 90)
@@
       (effects (font (size 1.27 1.27)) (justify right) hide)
     )
-    (property "Footprint" "easyeda_kicad:RES-TH_RK09K1130A6S" (id 2) (at 76.2 184.15 0)
+    (property "Footprint" "1_easyeda_kicad:RES-TH_RK09K1130A6S" (id 2) (at 76.2 184.15 0)
       (effects (font (size 1.27 1.27)) hide)
     )
@@
       (effects (font (size 1.27 1.27)) hide)
     )
-    (property "JLC Part" "Extended Part" (id 6) (at 49.53 105.41 0)
+    (property "JLC Part" "Extended Part" (id 7) (at 49.53 105.41 0)
       (effects (font (size 1.27 1.27)) hide)
     )
@@
     (pin "1")
   )
-  (symbol (lib_id "easyeda_kicad:RDC1022A05") (at 36.83 159.385 0) (mirror x) (unit 1)
+  (symbol (lib_id "1_easyeda_kicad:RDC1022A05") (at 36.83 159.385 0) (mirror x) (unit 1)
     (in_bom yes) (on_board yes) (fields_autoplaced)
     (property "Reference" "R1" (id 0) (at 39.37 159.3849 0)
@@
       (effects (font (size 1.27 1.27)) (justify left) hide)
     )
-    (property "Footprint" "easyeda_kicad:RES-ADJ-TH_RDC1022A05" (id 2) (at 36.83 146.685 0)
+    (property "Footprint" "1_easyeda_kicad:RES-ADJ-TH_RDC1022A05" (id 2) (at 36.83 146.685 0)
       (effects (font (size 1.27 1.27)) hide)
     )
@@
     (pin "1")
   )
-  (symbol (lib_id "easyeda_kicad:PEC11R-4220F-S0012") (at 66.04 158.75 0) (unit 1)
+  (symbol (lib_id "1_easyeda_kicad:PEC11R-4220F-S0012") (at 66.04 158.75 0) (unit 1)
     (in_bom yes) (on_board yes) (fields_autoplaced)
     (property "Reference" "SW13" (id 0) (at 66.04 148.59 0))
@@
       (effects (font (size 1.27 1.27)) hide)
     )
-    (property "Footprint" "easyeda_kicad:SW-TH_PEC11R-4220F-S0012" (id 2) (at 64.77 167.64 0)
+    (property "Footprint" "1_easyeda_kicad:SW-TH_PEC11R-4220F-S0012" (id 2) (at 64.77 167.64 0)
       (effects (font (size 1.27 1.27)) hide)
     )
@@
       (effects (font (size 1.27 1.27)) hide)
     )
-    (property "LCSC Part" "C143817" (id 4) (at 66.04 151.13 0))
+    (property "LCSC Part" "C143817" (id 4) (at 66.04 172.72 0))
     (pin "1")
     (pin "2")
@@
     (pin "4")
   )
-  (symbol (lib_id "easyeda_kicad:RDC1022A05") (at 36.83 181.61 0) (mirror x) (unit 1)
+  (symbol (lib_id "1_easyeda_kicad:RDC1022A05") (at 36.83 181.61 0) (mirror x) (unit 1)
     (in_bom yes) (on_board yes) (fields_autoplaced)
     (property "Reference" "R3" (id 0) (at 39.37 181.6099 0)
@@
       (effects (font (size 1.27 1.27)) (justify left) hide)
     )
-    (property "Footprint" "easyeda_kicad:RES-ADJ-TH_RDC1022A05" (id 2) (at 36.83 168.91 0)
+    (property "Footprint" "1_easyeda_kicad:RES-ADJ-TH_RDC1022A05" (id 2) (at 36.83 168.91 0)
       (effects (font (size 1.27 1.27)) hide)
     )
@@
     )
     (path "/3f780323-7f51-40a0-a137-fcfc16796bd7"
-      (reference "R1") (unit 1) (value "RDC1022A05") (footprint "easyeda_kicad:RES-ADJ-TH_RDC1022A05")
+      (reference "R1") (unit 1) (value "RDC1022A05") (footprint "1_easyeda_kicad:RES-ADJ-TH_RDC1022A05")
     )
     (path "/1de9b839-2ff9-4912-b4cc-5130ef7f4ed4"
-      (reference "R2") (unit 1) (value "RK09K1130A6S") (footprint "easyeda_kicad:RES-TH_RK09K1130A6S")
+      (reference "R2") (unit 1) (value "RK09K1130A6S") (footprint "1_easyeda_kicad:RES-TH_RK09K1130A6S")
     )
     (path "/cf1b2aae-5cc5-4bbf-b69a-f0a6e51bfff1"
-      (reference "R3") (unit 1) (value "RDC1022A05") (footprint "easyeda_kicad:RES-ADJ-TH_RDC1022A05")
+      (reference "R3") (unit 1) (value "RDC1022A05") (footprint "1_easyeda_kicad:RES-ADJ-TH_RDC1022A05")
     )
     (path "/efcc277a-7eb4-42da-8242-3b6924ff9ce9"
@@
     )
     (path "/42df5196-6128-450e-ba8a-a7c19bc9ea23"
-      (reference "SW13") (unit 1) (value "PEC11R-4220F-S0012") (footprint "easyeda_kicad:SW-TH_PEC11R-4220F-S0012")
+      (reference "SW13") (unit 1) (value "PEC11R-4220F-S0012") (footprint "1_easyeda_kicad:SW-TH_PEC11R-4220F-S0012")
     )
     (path "/aaa1dd85-7123-44ad-b089-9da9b7344d31"
